File: design/design_schematic/design_schematic.kicad_pcb (KiCad board)
At the start: 4 copper layers, 282.9 x 224.2 mm, 145 parts, among them IC2 XC9148G50CER-G, IC3 nRF52833-QDAA-R7, IC4 74AHCT125PW,118, IC5 MCP23018T-E_SS, IC6 XC9291B33D1R-G, J1 USB_C_Receptacle_USB2.0_16P, J2 Battery Pos, J3 Battery Neg, J4 OLED_128x32, J5 0781271220, U2 BQ24072RGT, U3 USB6B1, U4 BQ27441-G1, U5 PEC11L-4015F-S0015, U6 PEC11L-4015F-S0015, X1 32MHz

Commit message: no errors drc
Parts:
- added 3V3_2: TestPoint, TestPoint:TestPoint_Pad_D1.5mm, F.Cu at (84.7, 101.8)
- added 3v3_1: TestPoint, TestPoint:TestPoint_Pad_D1.5mm, F.Cu at (123.7, 93.9)
- added 5V_1: TestPoint, TestPoint:TestPoint_Pad_D1.5mm, F.Cu at (181.0, 67.5)
- added 5V_2: TestPoint, TestPoint:TestPoint_Pad_D1.5mm, F.Cu at (202.5, 91.5)
- added 5V_3: TestPoint, TestPoint:TestPoint_Pad_D1.5mm, F.Cu at (93.2, 46.3)
- added BAT_1: TestPoint, TestPoint:TestPoint_Pad_D1.5mm, F.Cu at (121.7, 103.5)
- added GND1: TestPoint, TestPoint:TestPoint_Pad_D1.5mm, F.Cu at (79.8, 29.2)
- added GND2: TestPoint, TestPoint:TestPoint_Pad_D1.5mm, F.Cu at (78.5, 91.1)
- added GND3: TestPoint, TestPoint:TestPoint_Pad_D1.5mm, F.Cu at (177.4, 30.2)
- added GND4: TestPoint, TestPoint:TestPoint_Pad_D1.5mm, F.Cu at (62.1, 108.9)
- added VBUS_1: TestPoint, TestPoint:TestPoint_Pad_D1.5mm, F.Cu at (82.6, 65.4)
- added VBUS_USB1: TestPoint, TestPoint:TestPoint_Pad_D1.5mm, F.Cu at (79.4, 32.6)
- C21, C24, C28, C29, C30, C31, C32, C33, C34, C5, C7, C8, C9: moved to B.Cu
- moved C13 165.6 mm to (201.7, 74.2), turned to 90 degrees
- moved C27 165.0 mm to (205.0, 58.6), turned to 90 degrees
- moved C26 163.6 mm to (203.9, 62.4), turned to -90 degrees
- moved C21 154.3 mm to (190.5, 81.8), turned to 180 degrees
- moved C29 148.4 mm to (188.2, 62.8), turned to 180 degrees
- moved C34 145.4 mm to (188.2, 43.7), turned to 180 degrees
- moved C31 114.4 mm to (152.5, 100.9), turned to 180 degrees
- moved C30 93.3 mm to (133.4, 81.9), turned to 180 degrees
- moved C28 88.8 mm to (128.7, 62.7), turned to 180 degrees
- moved C33 86.2 mm to (128.7, 43.7), turned to 180 degrees
- moved C9 78.3 mm to (104.5, 109.1)
- moved C5 73.6 mm to (89.8, 114.6)
- moved C1 71.4 mm to (85.5, 108.9), turned to 180 degrees
- moved C7 70.5 mm to (88.0, 116.9), turned to -90 degrees
- moved C24 70.5 mm to (92.3, 108.8)
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Connections:
- net Net-(F1-Pad1) renamed /VBUS_USB
- net Net-(J2-Pin_1) renamed /BAT
- net Net-(S26-NO) renamed /OUT
Routing:
- net /Row 0: track 122.0 -> 223.8 mm, vias 0 -> 8
- net 5V: track 34.4 -> 132.5 mm, vias 25 -> 32
- net /Row 1: track 119.3 -> 216.8 mm, vias 0 -> 8
- net /Row 3: track 126.1 -> 176.9 mm, vias 0 -> 2
- net GND: track 177.2 -> 227.8 mm, vias 94 -> 117
- net /Row 2: track 116.3 -> 165.0 mm, vias 0 -> 2
- net 3V3: track 239.7 -> 263.1 mm, vias 14 -> 16
- net Net-(IC2-BAT): track 26.2 -> 41.0 mm
- net /VBUS_USB: track 19.3 -> 24.9 mm, vias 0 -> 1
- net /BAT: track 139.3 -> 143.8 mm
- net /VBUS: track 137.2 -> 141.3 mm, vias 2 -> 3
- net /Column 5: track 202.3 -> 204.4 mm
- net /SDA: track 65.3 -> 63.5 mm
- net Net-(C15-Pad1): track 3.41 -> 4.27 mm
- net Net-(IC2-LX): track 3.72 -> 4.54 mm
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Other:
- board size 282.9 x 224.2 mm -> 147.4 x 95.2 mm

Commit message: routed no errors
Parts:
- removed C24: 100nF, ScottoKeebs_Components:Capacitor_0603
- added C37: 100nF, ScottoKeebs_Components:Capacitor_0603, F.Cu at (67.6, 98.5)
- added OUT1: TestPoint, TestPoint:TestPoint_Pad_D1.5mm, F.Cu at (81.8, 72.4)
- J5: value 0781271220 -> SFV12R-1STBE1HLF; footprint SamacSys_Parts:0781271220 -> SamacSys_Parts:SFV12R1STBE1HLF
- moved 5V_1 38.1 mm to (142.9, 68.2)
- moved J5 32.3 mm to (67.8, 90.7)
- moved C10 11.7 mm to (195.0, 65.9), turned to 180 degrees
- moved C27 7.99 mm to (201.4, 65.8), turned to 180 degrees
- moved 5V_2 4.79 mm to (200.7, 87.1)
- moved S26 4.63 mm to (198.0, 45.9)
- moved C25 4.33 mm to (199.3, 53.0)
- moved L6 3.47 mm to (198.9, 64.9)
- moved C26 3.24 mm to (200.6, 62.4)
- moved IC6 2.85 mm to (199.5, 67.9)
- moved L3 2.49 mm to (199.9, 72.1)
- moved IC2 2.40 mm to (199.9, 58.6)
- moved R12 2.29 mm to (79.2, 96.4), turned to 180 degrees
- moved IC4 2.06 mm to (85.0, 95.1)
- moved C13 1.94 mm to (199.8, 73.8), turned to 0 degrees
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Routing:
- net 5V: track 132.5 -> 114.5 mm, vias 32 -> 29
- net GND: track 227.8 -> 238.1 mm, vias 117 -> 116
- net /SDA: track 63.5 -> 73.0 mm, vias 3 -> 4
- net /OUT: track 164.9 -> 157.6 mm
- net /Row 3: track 176.9 -> 169.7 mm
- net /SCL: track 67.4 -> 73.3 mm, vias 0 -> 1
- net /Column 5: track 204.4 -> 202.1 mm
- net Net-(D1-DIN): track 57.3 -> 59.5 mm
- net /Column 4: track 229.6 -> 227.4 mm
- net 3V3: track 263.1 -> 260.9 mm, vias 16 -> 17
- net /CW2: track 74.8 -> 76.9 mm
- net /Row 0: track 223.8 -> 221.9 mm
- net /CCW2: track 80.1 -> 81.7 mm
- net Net-(D6-DOUT): track 151.1 -> 149.6 mm
- net /2A: track 46.3 -> 45.1 mm
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Other:
- board size 147.4 x 95.2 mm -> 144 x 95.2 mm

Commit message: uart switch
Parts:
- added REF**: MountingHole_3.2mm_M3, MountingHole:MountingHole_3.2mm_M3, F.Cu at (129.1, 113.5)
- added REF**: PinHeader_1x02_P1.00mm_Horizontal, Connector_PinHeader_1.00mm:PinHeader_1x02_P1.00mm_Horizontal, F.Cu at (40.2, 119.7)
- added REF**: MountingHole_3.2mm_M3, MountingHole:MountingHole_3.2mm_M3, F.Cu at (199.6, 35.9)
- added REF**: PinHeader_1x02_P1.00mm_Vertical, Connector_PinHeader_1.00mm:PinHeader_1x02_P1.00mm_Vertical, F.Cu at (43.3, 100.4)
- added REF**: PinHeader_1x04_P1.00mm_Horizontal, Connector_PinHeader_1.00mm:PinHeader_1x04_P1.00mm_Horizontal, F.Cu at (46.4, 116.9)
- added REF**: PinHeader_1x04_P1.00mm_Vertical, Connector_PinHeader_1.00mm:PinHeader_1x04_P1.00mm_Vertical, F.Cu at (43.7, 107.8)
- added REF**: MountingHole_3.2mm_M3, MountingHole:MountingHole_3.2mm_M3, F.Cu at (62.7, 78.6)
- added REF**: MountingHole_3.2mm_M3, MountingHole:MountingHole_3.2mm_M3, F.Cu at (62.9, 32.4)
Routing:
- net /Column 5: track 202.1 -> 199.3 mm
- net /Row 3: track 169.7 -> 168.3 mm
- net /BAT: track 143.8 -> 142.3 mm
