File: design/design_schematic/design_schematic.kicad_sch (KiCad schematic)
At the start: 158 parts, among them IC2 XC9148G50CER-G, IC3 nRF52833-QDAA-R7, IC4 74AHCT125PW,118, IC5 MCP23018T-E_SS, IC6 XC9291B33D1R-G, J1 USB_C_Receptacle_USB2.0_16P, J2 Battery Pos, J3 Battery Neg, J4 OLED_128x32, J5 SFV12R-1STBE1HLF, J6 Conn_01x04, U2 BQ24072RGT, U3 USB6B1, U4 BQ27441-G1, U5 PEC11L-4015F-S0015, U6 PEC11L-4015F-S0015, X1 32MHz

Commit message: production save prepare for left side
Parts:
- added 3V3_3: TestPoint, TestPoint:TestPoint_Pad_D1.5mm, symbol Connector:TestPoint
Connections:
- net 3V3: now also 3V3_3.1
Changed lines of the file:
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@@
 	(wire
 		(pts
+			(xy 304.8 171.45) (xy 304.8 175.26)
+		)
+		(stroke
+			(width 0)
+			(type default)
+		)
+	)
+	(wire
+		(pts
 			(xy 113.03 92.71) (xy 113.03 96.52)
 		)
@@
 	(wire
 		(pts
+			(xy 304.8 175.26) (xy 306.07 175.26)
+		)
+		(stroke
+			(width 0)
+			(type default)
+		)
+	)
+	(wire
+		(pts
 			(xy 105.41 93.98) (xy 105.41 92.71)
 		)
@@
 		)
 	)
+	(global_label "3V3"
+		(shape input)
+		(at 306.07 175.26 0)
+		(fields_autoplaced yes)
+		(effects
+			(font
+				(size 1.27 1.27)
+			)
+			(justify left)
+		)
+		(property "Intersheetrefs" "${INTERSHEET_REFS}"
+			(at 312.5628 175.26 0)
+			(effects
+				(font
+					(size 1.27 1.27)
+				)
+				(justify left)
+				(hide yes)
+			)
+		)
+	)
 	(symbol
 		(lib_id "power:GND")
@@
 					(unit 1)
 				)
+			)
+		)
+	)
+	(symbol
+		(lib_id "Connector:TestPoint")
+		(at 304.8 171.45 0)
+		(unit 1)
+		(exclude_from_sim no)
+		(in_bom yes)
+		(on_board yes)
+		(dnp no)
+		(fields_autoplaced yes)
+		(property "Reference" "3V3_3"
+			(at 307.34 166.8779 0)
+			(effects
+				(font
+					(size 1.27 1.27)
+				)
+				(justify left)
+			)
+		)
+		(property "Value" "TestPoint"
+			(at 307.34 169.4179 0)
+			(effects
+				(font
+					(size 1.27 1.27)
+				)
+				(justify left)
+			)
+		)
+		(property "Footprint" "TestPoint:TestPoint_Pad_D1.5mm"
+			(at 309.88 171.45 0)
+			(effects
+				(font
+					(size 1.27 1.27)
+				)
+				(hide yes)
+			)
+		)
+		(property "Datasheet" "~"
+			(at 309.88 171.45 0)
+			(effects
+				(font
+					(size 1.27 1.27)
+				)
+				(hide yes)
+			)
+		)
+		(property "Description" "test point"
+			(at 304.8 171.45 0)
+			(effects
+				(font
+					(size 1.27 1.27)
+				)
+				(hide yes)
+			)
+		)
+		(pin "1"
+		)
+		(instances
+			(project "design_schematic"
+				(path "/0454547d-f090-46a4-b0ab-f58aec48f156"
+					(reference "3V3_3")
+					(unit 1)
+				)
