File: design/rightside/rightside.kicad_sch (KiCad schematic)
At the start: 189 parts, among them IC2 XC9148G50CER-G, IC3 nRF52833-QDAA-R7, IC4 74AHCT125PW,118, IC5 MCP23018T-E_SS, IC6 XC9291B33D1R-G, J1 USB_C_Receptacle_USB2.0_16P, J2 Battery Pos, J3 Battery Neg, J4 OLED_128x32, J6 Conn_01x04, J7 F32Q-1A7H1-11012, U1 BQ27441-G1, U2 BQ24072RGT, U3 USB6B1, U5 PEC11L-4015F-S0015, U6 PEC11L-4015F-S0015, Y1 ECS-320-8-37B2-JTY-TR

Commit message: begin routing leftside
Changed lines of the file:
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@@
 	(polyline
 		(pts
-			(xy 580.39 13.97) (xy 580.39 241.3)
+			(xy 580.39 13.97) (xy 580.39 240.03)
 		)
 		(stroke
@@
 	(polyline
 		(pts
-			(xy 125.73 241.3) (xy 580.39 241.3)
-		)
-		(stroke
+			(xy 125.73 241.3) (xy 580.39 240.03)
+		)
+		(stroke
