File: design/leftside/leftside.kicad_pcb (KiCad board)
At the start: 4 copper layers, 142.6 x 96.2 mm, 221 parts, among them IC2 XC9148G50CER-G, IC3 nRF52833-QDAA-R7, IC4 74AHCT125PW,118, IC5 MCP23018T-E_SS, IC6 XC9291B33D1R-G, J1 USB_C_Receptacle_USB2.0_16P, J2 Battery Pos, J3 Battery Neg, J4 OLED_128x32, J6 Conn_01x04, J7 F32Q-1A7H1-11012, U1 BQ27441-G1, U2 BQ24072RGT, U3 USB6B1, U5 PEC11L-4015F-S0015, U6 PEC11L-4015F-S0015, Y1 ECS-320-8-37B2-JTY-TR

Commit message: setup nrf connect
Routing:
- net Net-(IC3-XC1): track 10.1 -> 11.2 mm
Changed lines of the file:
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@@
+	)
+	(segment
+		(start 146.7005 107.478399)
+		(end 146.074029 107.478399)
+		(width 0.2)
+		(layer "B.Cu")
+		(net 68)
+	)
+	(segment
+		(start 145.800932 107.751496)
+		(end 145.800932 107.751495)
+		(width 0.2)
+		(layer "B.Cu")
+		(net 68)
+	)
+	(segment
+		(start 145.782978 107.733541)
+		(end 145.800932 107.751495)
+		(width 0.2)
+		(layer "B.Cu")
+		(net 68)
 	)
 	(segment
@@
 		(width 0.2)
 		(layer "B.Cu")
+		(net 68)
+	)
+	(segment
+		(start 146.074029 107.478399)
+		(end 145.800932 107.751496)
+		(width 0.2)
+		(layer "B.Cu")
