File: design/leftside/leftside.kicad_sch (KiCad schematic)
At the start: 189 parts, among them IC2 XC9148G50CER-G, IC3 nRF52833-QDAA-R7, IC4 74AHCT125PW,118, IC5 MCP23018T-E_SS, IC6 XC9291B33D1R-G, J1 USB_C_Receptacle_USB2.0_16P, J2 Battery Pos, J3 Battery Neg, J4 OLED_128x32, J6 Conn_01x04, J7 F32Q-1A7H1-11012, U1 BQ27441-G1, U2 BQ24072RGT, U3 USB6B1, U5 PEC11L-4015F-S0015, U6 PEC11L-4015F-S0015, Y1 ECS-320-8-37B2-JTY-TR

Commit message: begin routing leftside
Connections:
- net GND: now also U5.MH1
- net OUT: now also S26.1 (COM); no longer S26.2 (NO)
- net at C10.1, C25.1, IC2.1 (BAT)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: now also S26.2 (NO); no longer S26.1 (COM)
- no-connect marks 34 -> 33
Other:
- moved on the sheet: S26
Changed lines of the file:
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@@
 	)
 	(no_connect
-		(at 161.29 219.71)
-	)
-	(no_connect
 		(at 86.36 171.45)
 	)
@@
 	(polyline
 		(pts
-			(xy 580.39 13.97) (xy 580.39 241.3)
+			(xy 580.39 13.97) (xy 580.39 240.03)
 		)
 		(stroke
@@
 	(polyline
 		(pts
-			(xy 125.73 241.3) (xy 580.39 241.3)
+			(xy 125.73 241.3) (xy 580.39 240.03)
 		)
 		(stroke
@@
 	(wire
 		(pts
-			(xy 262.89 97.79) (xy 262.89 99.06)
-		)
-		(stroke
-			(width 0)
-			(type default)
-		)
-	)
-	(wire
-		(pts
 			(xy 36.83 271.78) (xy 48.26 271.78)
 		)
@@
 	(wire
 		(pts
+			(xy 161.29 219.71) (xy 161.29 220.98)
+		)
+		(stroke
+			(width 0)
+			(type default)
+		)
+	)
+	(wire
+		(pts
 			(xy 500.38 41.91) (xy 500.38 43.18)
 		)
@@
 	(wire
 		(pts
+			(xy 260.35 96.52) (xy 260.35 97.79)
+		)
+		(stroke
+			(width 0)
+			(type default)
+		)
+	)
+	(wire
+		(pts
 			(xy 226.06 118.11) (xy 227.33 118.11)
 		)
@@
 	(wire
 		(pts
+			(xy 262.89 96.52) (xy 262.89 99.06)
+		)
+		(stroke
+			(width 0)
+			(type default)
+		)
+	)
+	(wire
+		(pts
 			(xy 312.42 135.89) (xy 313.69 135.89)
 		)
@@
 	)
 	(label "OUT"
-		(at 254 97.79 0)
+		(at 256.54 97.79 180)
 		(fields_autoplaced yes)
 		(effects
@@
 				(size 1.27 1.27)
 			)
-			(justify left bottom)
+			(justify right bottom)
 		)
 	)
@@
 	)
 	(symbol
+		(lib_id "power:GND")
+		(at 161.29 220.98 0)
+		(unit 1)
+		(exclude_from_sim no)
+		(in_bom yes)
+		(on_board yes)
+		(dnp no)
+		(fields_autoplaced yes)
+		(property "Reference" "#PWR0114"
+			(at 161.29 227.33 0)
+			(effects
+				(font
+					(size 1.27 1.27)
+				)
+				(hide yes)
+			)
+		)
+		(property "Value" "GND"
+			(at 161.29 226.06 0)
+			(effects
+				(font
+					(size 1.27 1.27)
+				)
+			)
+		)
+		(property "Footprint" ""
+			(at 161.29 220.98 0)
+			(effects
+				(font
+					(size 1.27 1.27)
+				)
+				(hide yes)
+			)
+		)
+		(property "Datasheet" ""
+			(at 161.29 220.98 0)
+			(effects
+				(font
+					(size 1.27 1.27)
+				)
+				(hide yes)
+			)
+		)
+		(property "Description" "Power symbol creates a global label with name \"GND\" , ground"
+			(at 161.29 220.98 0)
+			(effects
+				(font
+					(size 1.27 1.27)
+				)
+				(hide yes)
+			)
+		)
+		(pin "1"
+		)
+		(instances
+			(project "leftside"
+				(path "/0454547d-f090-46a4-b0ab-f58aec48f156"
+					(reference "#PWR0114")
+					(unit 1)
+				)
+			)
+		)
+	)
+	(symbol
 		(lib_id "ScottoKeebs:LED_SK6812MINI")
 		(at 474.98 50.8 0)
@@
 	(symbol
 		(lib_id "SamacSys_Parts:CL-SA-12C4-22")
-		(at 265.43 97.79 270)
-		(mirror x)
+		(at 257.81 96.52 90)
 		(unit 1)
 		(exclude_from_sim no)
@@
 		(dnp no)
 		(property "Reference" "S26"
-			(at 256.54 85.0899 90)
+			(at 266.7 83.8199 90)
 			(effects
 				(font
@@
 		)
 		(property "Value" "CL-SA-12C4-22"
-			(at 256.54 87.6299 90)
+			(at 266.7 86.3599 90)
 			(effects
 				(font
@@
 		)
 		(property "Footprint" "SamacSys_Parts:CLSA12C422"
-			(at 170.51 78.74 0)
+			(at 352.73 77.47 0)
 			(effects
 				(font
@@
 		)
 		(property "Datasheet" "https://www.nidec-components.com/e/catalog/switch/cl-sa.pdf"
-			(at 70.51 78.74 0)
+			(at 452.73 77.47 0)
 			(effects
 				(font
@@
 		)
 		(property "Description" "Slide Switches SPDT, ON-ON Slide, Red Actuator, 500mA @ 12V DC Right Angle PC Terminals, Bulk Packaging"
-			(at 265.43 97.79 0)
+			(at 257.81 96.52 0)
 			(effects
 				(font
@@
 		)
 		(property "Height" "2.54"
-			(at -129.49 78.74 0)
+			(at 652.73 77.47 0)
 			(effects
 				(font
@@
 		)
 		(property "Mouser Part Number" "229-CL-SA-12C4-22"
-			(at -229.49 78.74 0)
+			(at 752.73 77.47 0)
 			(effects
 				(font
@@
 		)
 		(property "Mouser Price/Stock" "https://www.mouser.co.uk/ProductDetail/Nidec-Components/CL-SA-12C4-22?qs=XeJtXLiO41QktpJxvsn9IA%3D%3D"
-			(at -329.49 78.74 0)
+			(at 852.73 77.47 0)
 			(effects
 				(font
@@
 		)
 		(property "Manufacturer_Name" "Nidec Copal"
-			(at -429.49 78.74 0)
+			(at 952.73 77.47 0)
 			(effects
 				(font
@@
 		)
 		(property "Manufacturer_Part_Number" "CL-SA-12C4-22"
-			(at -529.49 78.74 0)
+			(at 1052.73 77.47 0)
 			(effects
 				(font

Commit message: setup nrf connect
Parts:
- L5: value MCHK1608T1R0MKN -> 4.7uH
Other:
- moved on the sheet: C37, J7
