File: design/4layer/leftside/leftside.kicad_sch (KiCad schematic)
At the start: 189 parts, among them IC2 XC9148G50CER-G, IC3 nRF52833-QDAA-R7, IC4 74AHCT125PW,118, IC5 MCP23018T-E_SS, IC6 XC9291B33D1R-G, J1 USB_C_Receptacle_USB2.0_16P, J2 Battery Pos, J3 Battery Neg, J4 OLED_128x32, J6 Conn_01x04, J7 F32Q-1A7H1-11012, U1 BQ27441-G1, U2 BQ24072RGT, U3 USB6B1, U5 PEC11L-4015F-S0015, U6 PEC11L-4015F-S0015, Y1 ECS-320-8-37B2-JTY-TR

Commit message: New layout
Changed lines of the file:
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@@
 (kicad_sch
-	(version 20231120)
+	(version 20250114)
 	(generator "eeschema")
-	(generator_version "8.0")
+	(generator_version "9.0")
 	(paper "A1")
+	(rectangle
+		(start 213.36 78.74)
+		(end 285.75 142.24)
+		(stroke
+			(width 0)
+			(type dash)
+		)
+		(fill
+			(type none)
+		)
+	)
+	(rectangle
+		(start 143.51 81.28)
+		(end 210.82 137.16)
+		(stroke
+			(width 0)
+			(type dash)
+		)
+		(fill
+			(type none)
+		)
+	)
+	(rectangle
+		(start 287.02 40.64)
+		(end 354.33 147.32)
+		(stroke
+			(width 0)
+			(type dash)
+		)
+		(fill
+			(type none)
+		)
+	)
+	(text "Test Points"
+		(exclude_from_sim no)
+		(at 204.216 248.92 0)
+		(effects
+			(font
+				(size 5 5)
+				(thickness 1)
+				(bold yes)
+			)
+		)
+	)
+	(text "SK6803 LEDs"
+		(exclude_from_sim no)
+		(at 480.06 19.812 0)
+		(effects
+			(font
+				(size 5 5)
+				(thickness 1)
+				(bold yes)
+			)
+		)
+	)
+	(text "nRF52833 Module"
+		(exclude_from_sim no)
+		(at 70.612 28.194 0)
+		(effects
+			(font
+				(size 5 5)
+				(thickness 1)
+				(bold yes)
+			)
+		)
+	)
+	(text "GPIO Expander\n"
+		(exclude_from_sim no)
+		(at 71.12 215.646 0)
+		(effects
+			(font
+				(size 3 3)
+				(thickness 0.375)
+			)
+		)
+	)
+	(text "BLE Enabled\n"
+		(exclude_from_sim no)
+		(at 70.358 38.354 0)
+		(effects
+			(font
+				(size 3 3)
+				(thickness 0.375)
+			)
+		)
+	)
+	(text "DC-DC converter to turn variable input voltage to\nstable 3.3V/5V for load/LEDs. Battery fuel guage to\ndetermine battery percentage. 1uH for LX Step-Down results in\nlower ripple current and more stability. 10m Ohm resistor\nat 1% needed for precise columb counting for battery level sensing."
+		(exclude_from_sim no)
+		(at 336.296 157.226 0)
+		(effects
+			(font
+				(size 1 1)
+				(thickness 0.125)
+			)
+		)
+	)
+	(text "Power Management"
+		(exclude_from_sim no)
+		(at 248.412 22.606 0)
+		(effects
+			(font
+				(size 5 5)
+				(thickness 1)
+				(bold yes)
+			)
+		)
+	)
+	(text "Battery charging and USB power stage. Output 3.3V.\nILIM set to 3k, calculated by 1550/x where x is input current limit.\nISET set to 1.8k, calculated by 890/x where x is fast charge limit.\nx is set to 500mA to comply with USB standard."
+		(exclude_from_sim no)
+		(at 250.698 133.604 0)
+		(effects
+			(font
+				(size 1 1)
+				(thickness 0.125)
+			)
+		)
+	)
+	(text "USB-C and Data-line protection"
+		(exclude_from_sim no)
+		(at 194.818 133.858 0)
+		(effects
+			(font
+				(size 1 1)
+				(thickness 0.125)
+			)
+		)
+	)
+	(text "Peripherals\n"
+		(exclude_from_sim no)
+		(at 248.158 172.72 0)
+		(effects
+			(font
+				(size 5 5)
+				(thickness 1)
+				(bold yes)
+			)
+		)
+	)
+	(text "Switches\n"
+		(exclude_from_sim no)
+		(at 54.864 248.158 0)
+		(effects
+			(font
+				(size 5 5)
+				(thickness 1)
+				(bold yes)
+			)
+		)
+	)
+	(text "EC11 Encoders, OLED and Cirque glidepoint trackpad\n"
+		(exclude_from_sim no)
+		(at 248.158 179.832 0)
+		(effects
+			(font
+				(size 3 3)
+				(thickness 0.375)
+			)
+		)
+	)
+	(text "5V input and variable battery input changed to 3.3V output using 3.3V\nDC-DC Converter. Max. Current set to 500mA to match USB."
+		(exclude_from_sim no)
+		(at 223.52 153.67 0)
+		(effects
+			(font
+				(size 3 3)
+				(thickness 0.375)
+			)
+		)
+	)
+	(text "Contains USB C, ESD Protection, Battery charging/level sensing,\nand DC-DC conversion to 3.3V\n"
+		(exclude_from_sim no)
+		(at 250.19 33.528 0)
+		(effects
+			(font
+				(size 3 3)
+				(thickness 0.375)
+			)
+		)
+	)
+	(text "Uses logic shifter to bring 3.3V data input to 5V, uses MOSI SPI pin\nfor communication\n"
+		(exclude_from_sim no)
+		(at 479.552 29.21 0)
+		(effects
+			(font
+				(size 3 3)
+				(thickness 0.375)
+			)
+		)
+	)
+	(text "Stitching\nCapacitors"
+		(exclude_from_sim no)
+		(at 135.89 251.714 0)
+		(effects
+			(font
+				(size 5 5)
+				(thickness 1)
+				(bold yes)
+			)
+		)
+	)
 	(junction
 		(at 96.52 100.33)
@@
 		)
 	)
-	(rectangle
-		(start 213.36 78.74)
-		(end 285.75 142.24)
-		(stroke
-			(width 0)
-			(type dash)
-		)
-		(fill
-			(type none)
-		)
-	)
-	(rectangle
-		(start 143.51 81.28)
-		(end 210.82 137.16)
-		(stroke
-			(width 0)
-			(type dash)
-		)
-		(fill
-			(type none)
-		)
-	)
-	(rectangle
-		(start 287.02 40.64)
-		(end 354.33 147.32)
-		(stroke
-			(width 0)
-			(type dash)
-		)
-		(fill
-			(type none)
-		)
-	)
-	(text "Test Points"
-		(exclude_from_sim no)
-		(at 204.216 248.92 0)
-		(effects
-			(font
-				(size 5 5)
-				(thickness 1)
-				(bold yes)
-			)
-		)
-	)
-	(text "SK6803 LEDs"
-		(exclude_from_sim no)
-		(at 480.06 19.812 0)
-		(effects
-			(font
-				(size 5 5)
-				(thickness 1)
-				(bold yes)
-			)
-		)
-	)
-	(text "nRF52833 Module"
-		(exclude_from_sim no)
-		(at 70.612 28.194 0)
-		(effects
-			(font
-				(size 5 5)
-				(thickness 1)
-				(bold yes)
-			)
-		)
-	)
-	(text "GPIO Expander\n"
-		(exclude_from_sim no)
-		(at 71.12 215.646 0)
-		(effects
-			(font
-				(size 3 3)
-				(thickness 0.375)
-			)
-		)
-	)
-	(text "BLE Enabled\n"
-		(exclude_from_sim no)
-		(at 70.358 38.354 0)
-		(effects
-			(font
-				(size 3 3)
-				(thickness 0.375)
-			)
-		)
-	)
-	(text "DC-DC converter to turn variable input voltage to\nstable 3.3V/5V for load/LEDs. Battery fuel guage to\ndetermine battery percentage. 1uH for LX Step-Down results in\nlower ripple current and more stability. 10m Ohm resistor\nat 1% needed for precise columb counting for battery level sensing."
-		(exclude_from_sim no)
-		(at 336.296 157.226 0)
-		(effects
-			(font
-				(size 1 1)
-				(thickness 0.125)
-			)
-		)
-	)
-	(text "Power Management"
-		(exclude_from_sim no)
-		(at 248.412 22.606 0)
-		(effects
-			(font
-				(size 5 5)
-				(thickness 1)
-				(bold yes)
-			)
-		)
-	)
-	(text "Battery charging and USB power stage. Output 3.3V.\nILIM set to 3k, calculated by 1550/x where x is input current limit.\nISET set to 1.8k, calculated by 890/x where x is fast charge limit.\nx is set to 500mA to comply with USB standard."
-		(exclude_from_sim no)
-		(at 250.698 133.604 0)
-		(effects
-			(font
-				(size 1 1)
-				(thickness 0.125)
-			)
-		)
-	)
-	(text "USB-C and Data-line protection"
-		(exclude_from_sim no)
-		(at 194.818 133.858 0)
-		(effects
-			(font
-				(size 1 1)
-				(thickness 0.125)
-			)
-		)
-	)
-	(text "Peripherals\n"
-		(exclude_from_sim no)
-		(at 248.158 172.72 0)
-		(effects
-			(font
-				(size 5 5)
-				(thickness 1)
-				(bold yes)
-			)
-		)
-	)
-	(text "Switches\n"
-		(exclude_from_sim no)
-		(at 54.864 248.158 0)
-		(effects
-			(font
-				(size 5 5)
-				(thickness 1)
-				(bold yes)
-			)
-		)
-	)
-	(text "EC11 Encoders, OLED and Cirque glidepoint trackpad\n"
-		(exclude_from_sim no)
-		(at 248.158 179.832 0)
-		(effects
-			(font
-				(size 3 3)
-				(thickness 0.375)
-			)
-		)
-	)
-	(text "5V input and variable battery input changed to 3.3V output using 3.3V\nDC-DC Converter. Max. Current set to 500mA to match USB."
-		(exclude_from_sim no)
-		(at 223.52 153.67 0)
-		(effects
-			(font
-				(size 3 3)
-				(thickness 0.375)
-			)
-		)
-	)
-	(text "Contains USB C, ESD Protection, Battery charging/level sensing,\nand DC-DC conversion to 3.3V\n"
-		(exclude_from_sim no)
-		(at 250.19 33.528 0)
-		(effects
-			(font
-				(size 3 3)
-				(thickness 0.375)
-			)
-		)
-	)
-	(text "Uses logic shifter to bring 3.3V data input to 5V, uses MOSI SPI pin\nfor communication\n"
-		(exclude_from_sim no)
-		(at 479.552 29.21 0)
-		(effects
-			(font
-				(size 3 3)
-				(thickness 0.375)
-			)
-		)
-	)
-	(text "Stitching\nCapacitors"
-		(exclude_from_sim no)
-		(at 135.89 251.714 0)
-		(effects
-			(font
-				(size 5 5)
-				(thickness 1)
-				(bold yes)
-			)
-		)
-	)
 	(label "CW"
 		(at 57.15 148.59 180)
@@
 		)
 	)
+	(embedded_fonts no)
 )
