File: design/2layer/rightside/rightside.kicad_sch (KiCad schematic)
At the start: 189 parts, among them IC2 XC9148G50CER-G, IC3 nRF52833-QDAA-R7, IC4 74AHCT125PW,118, IC5 MCP23018T-E_SS, IC6 XC9291B33D1R-G, J1 USB_C_Receptacle_USB2.0_16P, J2 Battery Pos, J3 Battery Neg, J4 OLED_128x32, J6 Conn_01x04, J7 F32Q-1A7H1-11012, U1 BQ27441-G1, U2 BQ24072RGT, U3 USB6B1, U5 PEC11L-4015F-S0015, U6 PEC11L-4015F-S0015, Y1 ECS-320-8-37B2-JTY-TR

Commit message: LS two layer complete
Parts:
- removed 5V_2, 5V_3, 5V_5, BAT_1, GND4: TestPoint, TestPoint:TestPoint_Pad_D1.5mm, symbol Connector:TestPoint
- removed C20, C40, C46: 100nF, ScottoKeebs_Components:Capacitor_0603, symbol Device:C_Small
- removed IC4: 74AHCT125PW,118, SamacSys_Parts:SOP65P640X110-14N, symbol SamacSys_Parts:74AHCT125PW,118
- removed IC5: MCP23018T-E_SS, SamacSys_Parts:SOP65P780X200-24N, symbol SamacSys_Parts:MCP23018T-E_SS
- removed IC6: XC9291B33D1R-G, SamacSys_Parts:XC9290A07E1RG, symbol SamacSys_Parts:XC9291B33D1R-G
- removed L3: 1uH, Inductor_SMD:L_0603_1608Metric, symbol Device:L
- removed L5: MCHK1608T1R0MKN, INDC1608X80N, symbol SamacSys_Parts:MCHK1608T1R0MKN
- removed S26: CL-SA-12C4-22, SamacSys_Parts:CLSA12C422, symbol SamacSys_Parts:CL-SA-12C4-22
- added C47, C48: 4.7uF, ScottoKeebs_Components:Capacitor_0603, symbol Device:C_Small
- added CHG1, ~{PGOOD}1: TestPoint, TestPoint:TestPoint_Pad_D1.0mm, symbol Connector:TestPoint
- added IC1: XCL240B333FR-G, XCL103D503CRG, symbol SamacSys_Parts:XCL240B333FR-G
- added IC4: TCA9537DGSR, SOP50P490X110-10N, symbol SamacSys_Parts:TCA9537DGSR
- added IC6: TPS22917LDBVT, SOT95P280X145-6N, symbol SamacSys_Parts:TPS22917DBVT
- added IC7: SN74AHCT1G125DCKR, SOT65P210X110-5N, symbol SamacSys_Parts:SN74AHCT1G125DCKR
- added L3: 4.7uH, 1286ASH1R0MP2, symbol SamacSys_Parts:DFE201612E-4R7M=P2
- added LED1, LED2: White LED KW_EEL, KWEELP41RUS1U13K6L3X4X5R18, symbol SamacSys_Parts:KW_EELP41.RU-S1U1-3K6L-3X4X-5-R18
- added R11, R8: 270, Resistor_SMD:R_0603_1608Metric, symbol Device:R
- added R12: 10k, Resistor_SMD:R_0603_1608Metric, symbol Device:R
- added R13, R14: 4k7, Resistor_SMD:R_0603_1608Metric, symbol Device:R
- added R15, R16: 22, Resistor_SMD:R_0603_1608Metric, symbol Device:R
- added S25: CL-SA-12C4-22, SamacSys_Parts:CLSA12C422, symbol SamacSys_Parts:CL-SA-12C4-22
- C10: value 4.7uF -> 100pF
- C13: value 4.7uF -> 10uF
- C18: value 1uF -> 100nF; Notes Place close to gauge -> (none)
- J2: value Battery Pos -> Battery+
- J3: value Battery Neg -> Battery-
- R3: value 3k -> 540
- R4: value 1k8 -> 590
Connections:
- net 3V3: now also C13.1, C18.1, R9.1, IC1.3 (VOUT), IC1.8 (L2), IC4.10 (VCC), R12.1, R13.2, R14.2; no longer C13.2, R9.2
- net 5V: now also C47.1, IC1.4 (EN), IC1.6 (VIN), IC7.5 (VCC)
- net BAT: now also U1.7 (SRN), U2.2 (BAT), U2.3 (BAT), U2.5 (EN2), R11.1, R8.1; no longer C17.1, C18.1, J2.1 (Pin_1), U1.8 (SRP)
- net CCW: now also IC3.16 (P0.18); no longer IC3.15 (P0.17)
- net CCW2: now also IC3.14 (P0.15); no longer IC3.16 (P0.18)
- net CHG: now also CHG1.1, IC4.2 (P1), LED1.1 (K)
- net CW: now also IC3.17 (P0.20); no longer IC3.14 (P0.15)
- net CW2: now also IC3.15 (P0.17); no longer IC3.17 (P0.20)
- net D+: now also R16.2; no longer IC3.13 (D+)
- net D-: now also R15.1; no longer IC3.12 (D-)
- net GND: now also C13.2, C25.1, U2.6 (EN1), U5.MH1, U5.MH2, C47.2, C48.1, IC1.2 (AGND), IC1.5 (PGND), IC1.9 (EP), IC4.5 (GND), IC6.2 (GND), IC7.1 (~{OE}), IC7.3 (GND); no longer C10.2, C13.1, C25.2, U2.5 (EN2)
- net GPOUT: now also IC4.4 (P3), R12.2
- net INTA: now also IC4.7 (~{INT})
- net NO: now also IC4.3 (P2)
- net NO2: now also IC4.1 (P0)
- net OUT: now also C10.1, C48.2, IC6.1 (VIN), S25.1 (COM)
- net Row 0: now also IC3.7 (P0.11); no longer IC3.4 (P0.04)
- net Row 1: now also IC3.6 (P1.09); no longer IC3.5 (P0.05)
- net Row 2: now also IC3.5 (P0.05); no longer IC3.6 (P1.09)
- net Row 3: now also IC3.4 (P0.04); no longer IC3.7 (P0.11)
- net SCL: now also IC4.8 (SCL), R13.1
- net SDA: now also IC4.9 (SDA), R14.1
- net VBUS: no longer U2.6 (EN1)
- net at C14.1, IC3.29 (XC2): now also Y1.3 (OUT/IN); no longer Y1.1 (IN/OUT)
- net at C19.1, IC3.28 (XC1): now also Y1.1 (IN/OUT); no longer Y1.3 (OUT/IN)
- net at IC2.1 (BAT), IC2.3 (CE): now also C25.2, IC6.5 (QOD), IC6.6 (VOUT), L3.1; no longer C10.1, C25.1
- net at IC2.5 (LX): now also L3.2
- net at R10.1: now also IC7.4 (Y)
- net ~{PGOOD}: now reaches U2.7 (~{PGOOD})
- net ~{PGOOD}: now also LED2.1 (K), ~{PGOOD}1.1
- net 2A renamed A
- net A: now also IC7.2 (A)
- removed net BAT_SRN: R6.2, U1.7 (SRN), U2.2 (BAT), U2.3 (BAT)
- new net: IC6.3 (ON), S25.2 (NO)
- new net: C10.2, IC6.4 (CT)
- new net: LED2.2 (A), R11.2
- new net: IC1.1 (LX), IC1.7 (L1)
- new net: LED1.2 (A), R8.2
- new net: IC4.6 (~{RESET}), R9.2
- new net D2_N: IC3.12 (D-), R15.2
- new net D2_P: IC3.13 (D+), R16.1
- new net SRP: C17.1, J2.1 (Pin_1), R6.2, U1.8 (SRP)
- no-connect marks 34 -> 15
Other:
- note added: "Address: 0x2A (42)"
- note added: "Address: 0x3c (60)"
- note added: "Address: 0x49/73"
- note added: "Battery charging and USB power stage. Output 3.3V. ILIM controls input current limit calculated by 1550/R = limit. 3k = 500mA | 540 = 3A ISET controls battery current charge limit calculated by 890/R = limit. 1.8k = 500mA | 590 = 1.5A White LED for charging status with CHG. TPS2291 load switch for better stability when turning on/off. White LED for USB Power connection"
- note added: "DC-DC converters to turn variable battery voltage to stable 3.3V/5V for load/LEDs. Battery fuel guage to determine battery percentage. 10m Ohm resistor at 1% needed for precise columb counting for battery level sensing."
- note added: "GPIO Expander, EC11 Encoders, OLED and Cirque glidepoint trackpad"
- note removed: "Battery charging and USB power stage. Output 3.3V. ILIM set to 3k, calculated by 1550/x where x is input current limit. ISET set to 1.8k, calculated by 890/x where x is fast charge limit. x is set to 500mA to comply with USB standard."
- note removed: "DC-DC converter to turn variable input voltage to stable 3.3V/5V for load/LEDs. Battery fuel guage to determine battery percentage. 1uH for LX Step-Down results in lower ripple current and more stability. 10m Ohm resistor at 1% needed for precise columb counting for battery level sensing."
- note removed: "EC11 Encoders, OLED and Cirque glidepoint trackpad"
- note removed: "GPIO Expander"
- note removed: "Stitching Capacitors"
- moved on the sheet: 3V3_2, 3v3_1, 5V_1, 5V_4, ANT1, C1, C11, C12, C14, C15, C16, C17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

Commit message: place components for RS 2 layer
Parts:
- removed C27: 10uF-lowESR, ScottoKeebs_Components:Capacitor_0603, symbol Device:C_Small
- removed IC2: XC9148G50CER-G, SamacSys_Parts:XC9147_8_USP-6C, symbol SamacSys_Parts:XC9148G50CER-G
- removed L3: 4.7uH, 1286ASH1R0MP2, symbol SamacSys_Parts:DFE201612E-4R7M=P2
- added IC5: XCL110A503KR-G, XCL103D503CRG, symbol SamacSys_Parts:XCL110A503KR-G
- C26: value 10uF-lowESR -> 10uF
- F1: value 600mA -> 6A
Connections:
- net 5V: now also C26.2, IC5.6 (6/Vout); no longer C26.1
- net A: now also IC3.31 (P0.03); no longer IC3.23 (P0.10)
- net CCW: now also IC3.33 (P0.28); no longer IC3.16 (P0.18)
- net CCW2: now also IC3.35 (P0.30); no longer IC3.14 (P0.15)
- net CW: now also IC3.32 (P0.02); no longer IC3.17 (P0.20)
- net CW2: now also IC3.34 (P0.29); no longer IC3.15 (P0.17)
- net Column 0: now also IC3.22 (P0.09); no longer IC3.36 (P0.31)
- net Column 1: now also IC3.23 (P0.10); no longer IC3.35 (P0.30)
- net Column 2: now also IC3.14 (P0.15); no longer IC3.34 (P0.29)
- net Column 3: now also IC3.15 (P0.17); no longer IC3.33 (P0.28)
- net Column 4: now also IC3.16 (P0.18); no longer IC3.32 (P0.02)
- net Column 5: now also IC3.17 (P0.20); no longer IC3.31 (P0.03)
- net GND: now also C26.1, IC5.2 (2/AGND), IC5.4 (4/PGND), IC5.9 (9/EP); no longer C26.2
- net INTA: now also IC3.36 (P0.31); no longer IC3.22 (P0.09)
- net Row 0: now also IC3.4 (P0.04); no longer IC3.7 (P0.11)
- net Row 1: now also IC3.5 (P0.05); no longer IC3.6 (P1.09)
- net Row 2: now also IC3.6 (P1.09); no longer IC3.5 (P0.05)
- net Row 3: now also IC3.7 (P0.11); no longer IC3.4 (P0.04)
- net at C25.2, IC6.5 (QOD), IC6.6 (VOUT): now also IC5.1 (1/VIN), IC5.3 (3/EN), IC5.7 (7/L1)
- new net: IC5.5 (5/Lx), IC5.8 (8/L2)
Other:
- moved on the sheet: C25, C26

Commit message: prepare to add in EVQWGD001
Parts:
- added R17: 0, Resistor_SMD:R_0603_1608Metric, symbol Device:R
Connections:
- net CCW: now also IC3.32 (P0.02); no longer IC3.33 (P0.28)
- net CCW2: now also IC3.34 (P0.29); no longer IC3.35 (P0.30)
- net CHG: now also IC4.1 (P0); no longer IC4.2 (P1)
- net CW: now also IC3.33 (P0.28); no longer IC3.32 (P0.02)
- net CW2: now also IC3.35 (P0.30); no longer IC3.34 (P0.29)
- net NO2: now also IC4.2 (P1); no longer IC4.1 (P0)
- net Row 0: now also IC3.2 (P0.00); no longer IC3.4 (P0.04)
- net Row 1: now also IC3.3 (P0.01); no longer IC3.5 (P0.05)
- net Row 2: now also IC3.4 (P0.04); no longer IC3.6 (P1.09)
- net Row 3: now also IC3.5 (P0.05); no longer IC3.7 (P0.11)
- net SCL: now also IC3.6 (P1.09); no longer IC3.2 (P0.00)
- net SDA: now also IC3.7 (P0.11); no longer IC3.3 (P0.01)
- net VBUS: now also R17.1; no longer C2.2, IC3.10 (VBUS)
- new net: C2.2, IC3.10 (VBUS), R17.2
Other:
- moved on the sheet: C2, R13, R14

Commit message: New layout
Parts:
- removed U6: PEC11L-4015F-S0015, SamacSys_Parts:PEC11L4015FS0015, symbol SamacSys_Parts:PEC11L-4015F-S0015
- added EVQWGD1: ~, SamacSys_Parts:RollerEncoder_Panasonic_EVQWGD001, symbol SamacSys_Parts:EVQWGD001
Connections:
- net CCW2: now also EVQWGD1.B (CCW)
- net CW2: now also EVQWGD1.A (CW)
- net GND: now also EVQWGD1.C (COM), EVQWGD1.S2 (GND)
- net NO2: now also EVQWGD1.S1 (NO)
Other:
- note added: "DC-DC converters to turn variable battery voltage to stable 3.3V/5V for load/LEDs. Battery fuel gauge to determine battery percentage. 10m Ohm resistor at 1% needed for precise columb counting for battery level sensing."
- note removed: "DC-DC converters to turn variable battery voltage to stable 3.3V/5V for load/LEDs. Battery fuel guage to determine battery percentage. 10m Ohm resistor at 1% needed for precise columb counting for battery level sensing."

Commit message: RS begin to replace USB lines to shift 5V planes
Connections:
- net CCW2: now also IC3.5 (P0.05); no longer IC3.34 (P0.29)
- net CW2: now also IC3.4 (P0.04); no longer IC3.35 (P0.30)
- net Column 0: now also IC3.34 (P0.29); no longer IC3.22 (P0.09)
- net Column 1: now also IC3.22 (P0.09); no longer IC3.23 (P0.10)
- net GPOUT: now also IC4.3 (P2); no longer IC4.4 (P3)
- net INTA: now also IC3.3 (P0.01); no longer IC3.36 (P0.31)
- net NO: now also IC4.2 (P1); no longer IC4.3 (P2)
- net NO2: now also IC4.4 (P3); no longer IC4.2 (P1)
- net Row 0: now also IC3.35 (P0.30); no longer IC3.2 (P0.00)
- net Row 1: now also IC3.36 (P0.31); no longer IC3.3 (P0.01)
- net Row 2: now also IC3.23 (P0.10); no longer IC3.4 (P0.04)
- net Row 3: now also IC3.2 (P0.00); no longer IC3.5 (P0.05)
- net SCL: now also IC3.7 (P0.11), R14.1; no longer IC3.6 (P1.09), R13.1
- net SDA: now also IC3.6 (P1.09), R13.1; no longer IC3.7 (P0.11), R14.1
- net at D6.2 (DOUT): now also D14.4 (DIN); no longer D7.4 (DIN)
- net at D6.4 (DIN): now also D13.2 (DOUT); no longer D5.2 (DOUT)
- net at D28.2 (DOUT): now also D30.4 (DIN); no longer D29.4 (DIN)
- net at D29.2 (DOUT): now also D35.4 (DIN); no longer D30.4 (DIN)
- net at D34.2 (DOUT): now also D29.4 (DIN); no longer D35.4 (DIN)
- new net: D5.2 (DOUT), D7.4 (DIN)
Other:
- note added: "BLE Enabled - QFN40 Config 3"
- note removed: "BLE Enabled"
- moved on the sheet: D29, D35, D36, D6, R12
