File: design/2layer/rightside/rightside.kicad_sch (KiCad schematic)
At the start: 234 parts, among them IC2 MCP23009-E_MG, IC3 nRF52833-QDAA-R7, IC5 XCL110A503KR-G, IC6 TPS22917LDBVT, IC7 SN74AHCT1G125DCKR, IC8 TPS63051RMWT, J1 USB_C_Receptacle_USB2.0_16P, J2 Battery+, J3 Battery-, J4 OLED_128x32, J5 Conn_01x01, J6 Conn_01x04, J7 F32Q-1A7H1-11012, J8 Conn_01x01, U1 BQ27441-G1, U2 BQ24072RGT, U3 USB6B1, U5 PEC11L-4015F-S0015, Y1 ECS-320-8-37B2-JTY-TR

Commit message: RS LED wiring
Parts:
- removed D63: LED_SK6812MINI, ScottoKeebs_Components:LED_SK6812MINI, symbol ScottoKeebs:LED_SK6812MINI
Connections:
- net 5V: now also C2.2, C21.2, C28.2, C29.2, C3.2, C30.2, C31.2, C32.2, C33.2, C34.2, C35.2, C36.2, C38.2, C39.2, C4.2, C41.2, C42.2, C43.2, C44.2, C45.2; no longer C2.1, C21.1, C28.1, C29.1, C3.1, C30.1, C31.1, C32.1, C33.1, C34.1, C35.1, C36.1, C38.1, C39.1, C4.1, C41.1, C42.1, C43.1, C44.1, C45.1
- net GND: now also C2.1, C21.1, C28.1, C29.1, C3.1, C30.1, C31.1, C32.1, C33.1, C34.1, C35.1, C36.1, C38.1, C39.1, C4.1, C41.1, C42.1, C43.1, C44.1, C45.1; no longer C2.2, C21.2, C28.2, C29.2, C3.2, C30.2, C31.2, C32.2, C33.2, C34.2, C35.2, C36.2, C38.2, C39.2, C4.2, C41.2, C42.2, C43.2, C44.2, C45.2
- net Row 0: now also IC2.13 (GP4); no longer IC2.12 (GP3)
- net Row 1: now also IC2.15 (GP6); no longer IC2.13 (GP4)
- net Row 3: now also IC2.11 (GP2); no longer IC2.15 (GP6)
- net Row 4: now also IC2.12 (GP3); no longer IC2.16 (GP7)
- net Row 6: now also IC2.9 (GP0); no longer IC2.11 (GP2)
- net at D1.2 (DOUT): now also D2.4 (DIN)
- net at D1.4 (DIN): now also SR10.1; no longer D2.2 (DOUT)
- net at D39.2 (DOUT): now also D40.4 (DIN); no longer D38.4 (DIN)
- net at D39.4 (DIN): now also D38.2 (DOUT); no longer D40.2 (DOUT)
- net at D12.2 (DOUT): now also D13.4 (DIN); no longer D11.4 (DIN)
- net at D12.4 (DIN): now also D11.2 (DOUT); no longer D13.2 (DOUT)
- net at D61.2 (DOUT): now also D62.4 (DIN); no longer D9.4 (DIN)
- net at D61.4 (DIN): now also D60.2 (DOUT); no longer D62.2 (DOUT)
- net at D22.2 (DOUT): now also D23.4 (DIN); no longer D21.4 (DIN)
- net at D22.4 (DIN): now also D21.2 (DOUT); no longer D24.2 (DOUT)
- net at D4.2 (DOUT): now also D5.4 (DIN); no longer D3.4 (DIN)
- net at D4.4 (DIN): now also D3.2 (DOUT); no longer D48.2 (DOUT)
- net at D24.4 (DIN): now also D23.2 (DOUT); no longer D25.2 (DOUT)
- net at D41.2 (DOUT): now also D42.4 (DIN); no longer D40.4 (DIN)
- net at D9.2 (DOUT): now also D10.4 (DIN); no longer D8.4 (DIN)
- net at D57.4 (DIN): now also D56.2 (DOUT); no longer D50.2 (DOUT)
- net at D48.4 (DIN): now also D47.2 (DOUT); no longer D5.2 (DOUT)
- net at D6.2 (DOUT): now also D7.4 (DIN); no longer D5.4 (DIN)
- net at D6.4 (DIN): now also D5.2 (DOUT); no longer D7.2 (DOUT)
- net at D19.2 (DOUT): now also D20.4 (DIN); no longer D52.4 (DIN)
- net at D19.4 (DIN): now also D18.2 (DOUT); no longer D20.2 (DOUT)
- net at D41.4 (DIN): now also D40.2 (DOUT); no longer D42.2 (DOUT)
- net at D55.2 (DOUT): now also D56.4 (DIN); no longer D42.4 (DIN)
- net at D49.4 (DIN): now also D48.2 (DOUT); no longer SR10.1
- net at D35.2 (DOUT): now also D36.4 (DIN); no longer D34.4 (DIN)
- net at D35.4 (DIN): now also D34.2 (DOUT); no longer D36.2 (DOUT)
- net at D47.4 (DIN): now also D46.2 (DOUT); no longer D26.2 (DOUT)
- net at D30.2 (DOUT): now also D31.4 (DIN); no longer D29.4 (DIN)
- net at D30.4 (DIN): now also D29.2 (DOUT); no longer D53.2 (DOUT)
- net at D53.4 (DIN): now also D52.2 (DOUT); no longer D54.2 (DOUT)
- net at D17.2 (DOUT): now also D18.4 (DIN); no longer D16.4 (DIN)
- net at D17.4 (DIN): now also D16.2 (DOUT); no longer D18.2 (DOUT)
- net at D26.4 (DIN): now also D25.2 (DOUT); no longer D27.2 (DOUT)
- net at D33.4 (DIN): now also D32.2 (DOUT); no longer D34.2 (DOUT)
- net at D51.2 (DOUT): now also D52.4 (DIN); no longer D18.4 (DIN)
- net at D51.4 (DIN): now also D50.2 (DOUT); no longer D52.2 (DOUT)
- net at D37.2 (DOUT): now also D38.4 (DIN); no longer D36.4 (DIN)
- net at D25.4 (DIN): now also D24.2 (DOUT); no longer D23.2 (DOUT)
- net at D43.2 (DOUT): now also D44.4 (DIN); no longer D56.4 (DIN)
- net at D43.4 (DIN): now also D42.2 (DOUT); no longer D44.2 (DOUT)
- net at D54.4 (DIN): now also D53.2 (DOUT); no longer D31.2 (DOUT)
- net at D45.2 (DOUT): now also D46.4 (DIN); no longer D44.4 (DIN)
- net at D45.4 (DIN): now also D44.2 (DOUT); no longer D46.2 (DOUT)
- net at D28.4 (DIN): now also D27.2 (DOUT); no longer D29.2 (DOUT)
- net at D55.4 (DIN): now also D54.2 (DOUT); no longer D56.2 (DOUT)
- net at D37.4 (DIN): now also D36.2 (DOUT); no longer D38.2 (DOUT)
- net at D27.4 (DIN): now also D26.2 (DOUT); no longer D28.2 (DOUT)
- net at D59.2 (DOUT): now also D60.4 (DIN)
- net at D59.4 (DIN): now also D58.2 (DOUT); no longer D60.2 (DOUT)
- net at D8.2 (DOUT): now also D9.4 (DIN); no longer D10.4 (DIN)
- net at D14.2 (DOUT): now also D15.4 (DIN); no longer D13.4 (DIN)
- net at D14.4 (DIN): now also D13.2 (DOUT); no longer D15.2 (DOUT)
- net at D33.2 (DOUT): now also D34.4 (DIN); no longer D32.4 (DIN)
- net at D10.2 (DOUT): now also D11.4 (DIN); no longer D46.4 (DIN)
- new net: D20.2 (DOUT), D21.4 (DIN)
- new net: D2.2 (DOUT), D3.4 (DIN)
- new net: D31.2 (DOUT), D32.4 (DIN)
- new net: D7.2 (DOUT), D8.4 (DIN)
- new net: D28.2 (DOUT), D29.4 (DIN)
- new net: D15.2 (DOUT), D16.4 (DIN)
- no-connect marks 17 -> 16
Other:
- moved on the sheet: C2, C21, C28, C29, C3, C30, C31, C32, C33, C34, C35, C36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

Commit message: Fill all missing connections, except zone stitching vias
Parts:
- 3V3_2: footprint TestPoint:TestPoint_Pad_D1.5mm -> TestPoint:TestPoint_Pad_D1.0mm
Connections:
- net LED: now also IC3.35 (P0.30); no longer IC3.36 (P0.31)
- net NO2: now also IC3.36 (P0.31); no longer IC3.35 (P0.30)
Changed lines of the file:
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@@
 	)
 	(label "NO2"
-		(at 64.77 54.61 0)
+		(at 62.23 52.07 0)
 		(effects
 			(font
@@
 	)
 	(label "LED"
-		(at 62.23 52.07 0)
+		(at 64.77 54.61 0)
 		(effects
 			(font
@@
 			)
 		)
-		(property "Footprint" "TestPoint:TestPoint_Pad_D1.5mm"
+		(property "Footprint" "TestPoint:TestPoint_Pad_D1.0mm"
 			(at 100.33 360.68 0)
 			(hide yes)
