File: design/2layer/leftside/leftside.kicad_sch (KiCad schematic)
At the start: 237 parts, among them IC2 MCP23009-E_MG, IC3 nRF52833-QDAA-R7, IC5 XCL110A503KR-G, IC6 TPS22917LDBVT, IC7 SN74AHCT1G125DCKR, IC8 TPS63051RMWT, J1 USB_C_Receptacle_USB2.0_16P, J2 Battery+, J3 Battery-, J4 OLED_128x32, J5 Conn_01x01, J6 Conn_01x04, J7 F32Q-1A7H1-11012, J8 Conn_01x01, U1 BQ27441-G1, U2 BQ24072RGT, U3 USB6B1, U5 PEC11L-4015F-S0015, Y1 ECS-320-8-37B2-JTY-TR

Commit message: LS Kicad 10 migration
Parts:
- removed VBUS_USB1: TestPoint, TestPoint:TestPoint_Pad_D1.0mm, symbol Connector:TestPoint
- EVQWGD1: value ~ -> (none)
Connections:
- net at D49.4 (DIN): now also SR10.1; no longer SR10.2
- net at IC7.4 (Y): now also SR10.2; no longer SR10.1
Other:
- moved on the sheet: 3V3_2, 5V_1, 5V_4, C2, C21, C28, C29, C3, C30, C31, C32, C33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
